File: FAN.kicad_sch (KiCad schematic)
At the start: 4 parts, among them J17 Molex 470531000, U11 EMC2301-1-ACZL-TR

Commit message: added 3D models
Parts:
- J17: footprint Connector:FanPinHeader_1x04_P2.54mm_Vertical -> Connector_Wire:SolderWirePad_1x01_SMD_1x2mm
Changed lines of the file:
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@@
   (junction (at 106.68 140.97) (diameter 1.016) (color 0 0 0 0))
   (junction (at 144.78 140.97) (diameter 1.016) (color 0 0 0 0))
+  (no_connect (at 138.43 138.43))
   (no_connect (at 138.43 135.89))
-  (no_connect (at 138.43 138.43))
   (wire (pts (xy 102.87 125.73) (xy 144.78 125.73))
     (stroke (width 0) (type solid) (color 0 0 0 0))
@@
       (effects (font (size 1.27 1.27)) (justify left))
     )
-    (property "Footprint" "Connector:FanPinHeader_1x04_P2.54mm_Vertical" (id 2) (at 184.15 137.16 0)
-      (effects (font (size 1.27 1.27)) hide)
-    )
+    (property "Footprint" "Connector_Wire:SolderWirePad_1x01_SMD_1x2mm" (id 2) (at 184.15 137.16 0)
+      (effects (font (size 1.27 1.27)) hide)
+    )
