File: PSUs.kicad_sch (KiCad schematic)
At the start: 23 parts, among them J19 XT30, Q1 DMP3013SFV-7, U8 LMR33640DDDAR

Commit message: library management
Parts:
- C18, C22: footprint (none) -> Capacitor_SMD:C_1210_3225Metric
- C24, C31: footprint (none) -> Capacitor_SMD:C_0603_1608Metric
- C25, C26, C27: footprint (none) -> Capacitor_SMD:C_0402_1005Metric
- C28, C29, C30: footprint (none) -> Capacitor_SMD:C_0805_2012Metric
- L1: footprint (none) -> Open-HD:IND_XAL6060-472MEB
- R19, R4, R9: footprint (none) -> Resistor_SMD:R_0402_1005Metric
- U8: footprint (none) -> Open-HD:NOPB
Changed lines of the file:
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@@
     (property "Reference" "L1" (id 0) (at 160.02 113.03 90))
     (property "Value" "4.7uH" (id 1) (at 160.02 115.57 90))
-    (property "Footprint" "" (id 2) (at 160.02 118.11 0)
+    (property "Footprint" "Open-HD:IND_XAL6060-472MEB" (id 2) (at 160.02 118.11 0)
       (effects (font (size 1.27 1.27)) hide)
     )
@@
     (property "Reference" "R4" (id 0) (at 147.32 120.65 90))
     (property "Value" "100k" (id 1) (at 147.32 125.73 90))
-    (property "Footprint" "" (id 2) (at 147.32 124.968 90)
+    (property "Footprint" "Resistor_SMD:R_0402_1005Metric" (id 2) (at 147.32 124.968 90)
       (effects (font (size 1.27 1.27)) hide)
     )
@@
       (effects (font (size 1.27 1.27)) (justify left))
     )
-    (property "Footprint" "" (id 2) (at 181.102 121.92 90)
+    (property "Footprint" "Resistor_SMD:R_0402_1005Metric" (id 2) (at 181.102 121.92 90)
       (effects (font (size 1.27 1.27)) hide)
     )
@@
       (effects (font (size 1.27 1.27)) (justify left))
     )
-    (property "Footprint" "" (id 2) (at 181.102 133.35 90)
+    (property "Footprint" "Resistor_SMD:R_0402_1005Metric" (id 2) (at 181.102 133.35 90)
       (effects (font (size 1.27 1.27)) hide)
     )
@@
       (effects (font (size 1.27 1.27)) (justify left))
     )
-    (property "Footprint" "" (id 2) (at 72.0852 123.19 0)
+    (property "Footprint" "Capacitor_SMD:C_1210_3225Metric" (id 2) (at 72.0852 123.19 0)
       (effects (font (size 1.27 1.27)) hide)
     )
@@
       (effects (font (size 1.27 1.27)) (justify left))
     )
-    (property "Footprint" "" (id 2) (at 84.7852 123.19 0)
+    (property "Footprint" "Capacitor_SMD:C_1210_3225Metric" (id 2) (at 84.7852 123.19 0)
       (effects (font (size 1.27 1.27)) hide)
     )
@@
       (effects (font (size 1.27 1.27)) (justify left))
     )
-    (property "Footprint" "" (id 2) (at 96.2152 123.19 0)
+    (property "Footprint" "Capacitor_SMD:C_0603_1608Metric" (id 2) (at 96.2152 123.19 0)
       (effects (font (size 1.27 1.27)) hide)
     )
@@
       (effects (font (size 1.27 1.27)) (justify left))
     )
-    (property "Footprint" "" (id 2) (at 107.6452 135.89 0)
+    (property "Footprint" "Capacitor_SMD:C_0402_1005Metric" (id 2) (at 107.6452 135.89 0)
       (effects (font (size 1.27 1.27)) hide)
     )
@@
       (effects (font (size 1.27 1.27)) (justify left))
     )
-    (property "Footprint" "" (id 2) (at 147.0152 115.57 0)
+    (property "Footprint" "Capacitor_SMD:C_0402_1005Metric" (id 2) (at 147.0152 115.57 0)
       (effects (font (size 1.27 1.27)) hide)
     )
@@
       (effects (font (size 1.27 1.27)) (justify left))
     )
-    (property "Footprint" "" (id 2) (at 173.6852 127 0)
+    (property "Footprint" "Capacitor_SMD:C_0402_1005Metric" (id 2) (at 173.6852 127 0)
       (effects (font (size 1.27 1.27)) hide)
     )
@@
       (effects (font (size 1.27 1.27)) (justify left))
     )
-    (property "Footprint" "" (id 2) (at 197.8152 128.27 0)
+    (property "Footprint" "Capacitor_SMD:C_0805_2012Metric" (id 2) (at 197.8152 128.27 0)
       (effects (font (size 1.27 1.27)) hide)
     )
@@
       (effects (font (size 1.27 1.27)) (justify left))
     )
-    (property "Footprint" "" (id 2) (at 209.2452 128.27 0)
+    (property "Footprint" "Capacitor_SMD:C_0805_2012Metric" (id 2) (at 209.2452 128.27 0)
       (effects (font (size 1.27 1.27)) hide)
     )
@@
       (effects (font (size 1.27 1.27)) (justify left))
     )
-    (property "Footprint" "" (id 2) (at 219.4052 128.27 0)
+    (property "Footprint" "Capacitor_SMD:C_0805_2012Metric" (id 2) (at 219.4052 128.27 0)
       (effects (font (size 1.27 1.27)) hide)
     )
@@
       (effects (font (size 1.27 1.27)) (justify left))
     )
-    (property "Footprint" "" (id 2) (at 229.5652 128.27 0)
+    (property "Footprint" "Capacitor_SMD:C_0603_1608Metric" (id 2) (at 229.5652 128.27 0)
       (effects (font (size 1.27 1.27)) hide)
     )
@@
     (property "Reference" "U8" (id 0) (at 125.73 105.41 0))
     (property "Value" "LMR33640DDDAR" (id 1) (at 125.73 107.95 0))
-    (property "Footprint" "" (id 2) (at 116.84 106.68 0)
-      (effects (font (size 1.27 1.27)) hide)
-    )
+    (property "Footprint" "Open-HD:NOPB" (id 2) (at 116.84 106.68 0)
+      (effects (font (size 1.27 1.27)) hide)
+    )

Commit message: added 3D models
Parts:
- J19: footprint XT-30:AMASS_XT30PW-M_1x02_P2.50mm_Horizontal -> Open-HD:AMASS_XT30PW-M_1x02_P2.50mm_Horizontal
Changed lines of the file:
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@@
     (property "Reference" "J19" (id 0) (at 59.69 39.37 0))
     (property "Value" "XT30" (id 1) (at 59.69 41.91 0))
-    (property "Footprint" "XT-30:AMASS_XT30PW-M_1x02_P2.50mm_Horizontal" (id 2) (at 62.23 43.18 0)
+    (property "Footprint" "Open-HD:AMASS_XT30PW-M_1x02_P2.50mm_Horizontal" (id 2) (at 62.23 43.18 0)
       (effects (font (size 1.27 1.27)) hide)
     )
