File: CM4_Carrier.kicad_pcb (KiCad board)
At the start: 4 copper layers, 112 parts, among them J1 Conn_01x03, J10 Conn_01x20, J11 USB_OTG, J12 10018783-11200TLF, J13 BM04B-GHS-TBT(LF)(SN)(N), J14 BM04B-GHS-TBT(LF)(SN)(N), J15 Conn_01x22_Female, J17 Molex 470531000, J18 BM04B-GHS-TBT(LF)(SN)(N), J19 XT30, J2 Conn_02x07_Odd_Even, J21 BM04B-GHS-TBT(LF)(SN)(N), J3 Conn_01x03, J4 DF40C-24DP-0.4V_51_, J5 DF40C-24DP-0.4V_51_, J6 THD-02-R, J7 Micro_SD_Card_Det, J8 HDMI_D_1.4, J9 Conn_02x08_Odd_Even, Q1 DMP3013SFV-7, U1 TPD4EUSB30, U10 AP22653W6, U11 EMC2301-1-ACZL-TR, U12 RT9742SNGV, U13 FSUSB42MUX, U18 RT9742GGJ5, U2 TPD4EUSB30, U4 TPD4EUSB30, U5 74LVC1G07SE-7, U6 USB2514B-I/M2, U7 AP22653W6, U8 LMR33640DDDAR, U9 74LVC1G07SE-7, Y1 24MHz

Commit message: starting to lay out switching regulator
Parts:
- removed C36: 100n 100v, Capacitor_SMD:C_0402_1005Metric
- removed C40: 100n, Capacitor_SMD:C_0402_1005Metric
- removed D4: MMBZ5242BLT3G, Diode_SMD:D_SOT-23_ANK
- removed J19: XT30, Open-HD:AMASS_XT30PW-M_1x02_P2.50mm_Horizontal
- removed J4, J5: DF40C-24DP-0.4V_51_, Open-HD:DF40C24DP04V51
- removed R26: 12K 1%, Resistor_SMD:R_0402_1005Metric
- removed U8: LMR33640DDDAR, Open-HD:NOPB
- added C32: 22uF, Capacitor_SMD:C_0805_2012Metric, F.Cu at (137.4, 61.7)
- added C33: 100nF, Capacitor_SMD:C_0603_1608Metric, F.Cu at (125.0, 39.9)
- added D3: MMBZ5242BLT3G, Diode_SMD:D_SOT-23_ANK, B.Cu at (138.6, 71.4)
- added J16: XT30, Open-HD:AMASS_XT30PW-M_1x02_P2.50mm_Horizontal, F.Cu at (149.2, 67.4)
- added JP1: Jumper, Jumper:SolderJumper-2_P1.3mm_Bridged_RoundedPad1.0x1.5mm, F.Cu at (218.2, 147.4)
- added JP2: Jumper, Jumper:SolderJumper-2_P1.3mm_Bridged_RoundedPad1.0x1.5mm, F.Cu at (223.6, 138.9)
- added JP3: Jumper_NC_Dual, Jumper:SolderJumper-3_P1.3mm_Bridged12_RoundedPad1.0x1.5mm, F.Cu at (213.2, 147.4)
- added SW1: SW_SPST, Button_Switch_SMD:SW_SPST_B3S-1000, F.Cu at (215.9, 141.4)
- added U3: LMR33640DDDAR, Open-HD:NOPB, F.Cu at (126.4, 66.8)
- C24: value 220nF -> 100n 100v; footprint Capacitor_SMD:C_0603_1608Metric -> Capacitor_SMD:C_0402_1005Metric
- C25: value 1uF -> 220nF; footprint Capacitor_SMD:C_0402_1005Metric -> Capacitor_SMD:C_0603_1608Metric
- C26: value 100nF -> 1uF
- C27: value 10pF -> 100n
- C28: value 22uF -> 100nF; footprint Capacitor_SMD:C_0805_2012Metric -> Capacitor_SMD:C_0402_1005Metric
- C29: value 22uF -> 10pF; footprint Capacitor_SMD:C_0805_2012Metric -> Capacitor_SMD:C_0402_1005Metric
- C31: value 100nF -> 22uF; footprint Capacitor_SMD:C_0603_1608Metric -> Capacitor_SMD:C_0805_2012Metric
- J1: value Conn_01x03 -> Conn_01x22_Female; footprint Connector_PinHeader_2.54mm:PinHeader_1x03_P2.54mm_Vertical -> Connector_FFC-FPC:Hirose_FH12-22S-0.5SH_1x22-1MP_P0.50mm_Horizontal; moved to B.Cu
- J11, J7, R17, R18, R29, U18: moved to B.Cu
- J2: value Conn_02x07_Odd_Even -> Conn_01x22_Female; footprint Connector_PinHeader_2.54mm:PinHeader_2x07_P2.54mm_Vertical -> Connector_FFC-FPC:Hirose_FH12-22S-0.5SH_1x22-1MP_P0.50mm_Horizontal
- R4: value 100k -> 12K 1%; moved to B.Cu
- moved J1 187.3 mm to (128.2, 135.8), turned to 180 degrees
- moved C12 186.2 mm to (70.9, 87.6)
- moved C13 186.2 mm to (76.4, 87.7)
- moved D1 186.2 mm to (72.1, 97.0)
- moved D2 186.2 mm to (75.7, 97.0)
- moved R1 186.2 mm to (75.2, 94.5)
- moved R10 186.2 mm to (73.0, 94.5)
- moved TP3 186.2 mm to (75.8, 94.2)
- moved TP5 186.2 mm to (72.5, 94.2)
- moved U12 186.2 mm to (73.5, 87.4)
- moved U5 186.2 mm to (75.0, 91.4)
- moved J2 85.4 mm to (128.2, 135.8), turned to 0 degrees
- moved J12 70.6 mm to (204.6, 112.2), turned to 0 degrees
- moved J7 64.5 mm to (152.2, 110.4), turned to -90 degrees
- moved R18 53.6 mm to (162.5, 107.8), turned to 180 degrees
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Connections:
- net /FAN/SCL renamed /Power/SCL
- net /FAN/SDA renamed /Power/SDA
- C18 pad 1: /PSUs/+12v -> /Power/+12v
- C22 pad 1: /PSUs/+12v -> /Power/+12v
- C24 pad 1: /PSUs/+12v -> Net-(C24-Pad1)
- C25 pad 1: Net-(C25-Pad1) -> /Power/+12v
- C26 pad 2: Net-(C26-Pad2) -> GND
- C27 pad 1: /+5v -> /Power/+12v
- C28 pad 1: /+5v -> Net-(C28-Pad1)
- C28 pad 2: GND -> Net-(C28-Pad2)
- C29 pad 2: GND -> Net-(C29-Pad2)
- J1 pad 1: /GLOBAL_EN -> GND
- J1 pad 2: GND -> /CM4_HighSpeed/CAM0_D0_N
- J1 pad 3: /CM4_GPIO ( Ethernet, GPIO, SDCARD)/RUN_PG -> /CM4_HighSpeed/CAM0_D0_P
- J2 pad 11: /TV_OUT -> /CM4_HighSpeed/CAM1_D2_N
- J2 pad 12: GND -> /CM4_HighSpeed/CAM1_D2_P
- J2 pad 13: Net-(J2-Pad13) -> GND
- J2 pad 14: /GLOBAL_EN -> /CM4_HighSpeed/CAM1_D3_N
- J2 pad 2: /CM4_GPIO ( Ethernet, GPIO, SDCARD)/nRPIBOOT -> /CM4_HighSpeed/CAM1_D0_N
- J2 pad 3: GND -> /CM4_HighSpeed/CAM1_D0_P
- J2 pad 4: /CM4_GPIO ( Ethernet, GPIO, SDCARD)/EEPROM_nWP -> GND
- J2 pad 5: /CM4_GPIO ( Ethernet, GPIO, SDCARD)/AIN0 -> /CM4_HighSpeed/CAM1_D1_N
- J2 pad 6: /CM4_GPIO ( Ethernet, GPIO, SDCARD)/AIN1 -> /CM4_HighSpeed/CAM1_D1_P
- J2 pad 8: /CM4_GPIO ( Ethernet, GPIO, SDCARD)/SYNC_IN -> /CM4_HighSpeed/CAM1_C_N
- J2 pad 9: /CM4_GPIO ( Ethernet, GPIO, SDCARD)/SYNC_OUT -> /CM4_HighSpeed/CAM1_C_P
- L1 pad 1: Net-(C26-Pad2) -> Net-(C28-Pad2)
- Module1 pad 99: /GLOBAL_EN -> /CM4_GPIO ( Ethernet, GPIO, SDCARD)/GLOBAL_EN
- Q1 pad 1: /PSUs/+12v -> /Power/+12v
- Q1 pad 2: /PSUs/+12v -> /Power/+12v
- Q1 pad 3: /PSUs/+12v -> /Power/+12v
- Q1 pad 4: Net-(C40-Pad2) -> Net-(C27-Pad2)
- Q1 pad 5: Net-(C36-Pad1) -> Net-(C24-Pad1)
- R19 pad 1: Net-(C27-Pad2) -> Net-(C29-Pad2)
- R4 pad 1: Net-(R4-Pad1) -> Net-(C27-Pad2)
- R4 pad 2: /+5v -> GND
- R9 pad 2: Net-(C27-Pad2) -> Net-(C29-Pad2)
- U9 pad 4: Net-(J2-Pad13) -> Net-(U9-Pad4)
Routing:
- net Net-(C27-Pad2): track 0.00 -> 5.59 mm, vias 0 -> 1
- net Net-(C24-Pad1): vias 0 -> 14
- net /Power/+12v: vias 0 -> 19
- added copper zone on B.Cu, net /Power/+12v
- added copper zone on F.Cu, net /Power/+12v
- added copper zone on In1.Cu, net /Power/+12v
- added copper zone on In2.Cu, net /Power/+12v
- added copper zone on B.Cu, net Net-(C24-Pad1)
- added copper zone on F.Cu, net Net-(C24-Pad1)
- added copper zone on In1.Cu, net Net-(C24-Pad1)
- added copper zone on In2.Cu, net Net-(C24-Pad1)
Other:
- board outline added: 47 x 86 mm
- board text removed: "Ethernet"

Commit message: cleanup
Parts:
- moved C12 23.6 mm to (64.8, 110.4)
- moved C13 23.6 mm to (70.2, 110.5)
- moved D1 23.6 mm to (65.9, 119.8)
- moved D2 23.6 mm to (69.5, 119.8)
- moved R1 23.6 mm to (69.0, 117.3)
- moved R10 23.6 mm to (66.8, 117.3)
- moved TP3 23.6 mm to (69.6, 117.0)
- moved TP5 23.6 mm to (66.3, 117.0)
- moved U12 23.6 mm to (67.3, 110.2)
- moved U5 23.6 mm to (68.8, 114.2)
- moved C28 0.20 mm to (125.2, 62.6)
Routing:
- net Net-(C28-Pad1): track 0.00 -> 1.54 mm
- net Net-(C28-Pad2): track 0.00 -> 0.12 mm, vias 0 -> 8
- added copper zone on B.Cu, net Net-(C28-Pad2)
- added copper zone on F.Cu, net Net-(C28-Pad2)
- added copper zone on In1.Cu, net Net-(C28-Pad2)
- added copper zone on In2.Cu, net Net-(C28-Pad2)
Other:
- board text added: "Place jumpers and buttons here ->"
Changed lines of the file:
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@@
   (net 234 "Net-(J10-Pad19)")
   (module "Capacitor_SMD:C_0402_1005Metric" (layer "F.Cu")
-    (at 70.942394 87.624 90)
+    (at 64.75 110.4 90)
     (descr "Capacitor SMD 0402 (1005 Metric), square (rectangular) end terminal, IPC_7351 nominal, (Body size source: http://www.tortai-tech.com/upload/download/2011102023233369053.pdf), generated with kicad-footprint-generator")
     (tags "capacitor")
@@
   )
   (module "Capacitor_SMD:C_0402_1005Metric" (layer "F.Cu")
-    (at 76.392394 87.724 90)
+    (at 70.2 110.5 90)
     (descr "Capacitor SMD 0402 (1005 Metric), square (rectangular) end terminal, IPC_7351 nominal, (Body size source: http://www.tortai-tech.com/upload/download/2011102023233369053.pdf), generated with kicad-footprint-generator")
     (tags "capacitor")
@@
   )
   (module "Resistor_SMD:R_0402_1005Metric" (layer "F.Cu")
-    (at 72.992394 94.524 90)
+    (at 66.8 117.3 90)
     (descr "Resistor SMD 0402 (1005 Metric), square (rectangular) end terminal, IPC_7351 nominal, (Body size source: http://www.tortai-tech.com/upload/download/2011102023233369053.pdf), generated with kicad-footprint-generator")
     (tags "resistor")
@@
   )
   (module "Package_TO_SOT_SMD:SOT-23" (layer "F.Cu")
-    (at 73.492394 87.424 90)
+    (at 67.3 110.2 90)
     (descr "SOT-23, Standard")
     (tags "SOT-23")
@@
   )
   (module "LED_SMD:LED_0603_1608Metric" (layer "F.Cu")
-    (at 75.742394 97.024 180)
+    (at 69.55 119.8 180)
     (descr "LED SMD 0603 (1608 Metric), square (rectangular) end terminal, IPC_7351 nominal, (Body size source: http://www.tortai-tech.com/upload/download/2011102023233369053.pdf), generated with kicad-footprint-generator")
     (tags "diode")
@@
   )
   (module "LED_SMD:LED_0603_1608Metric" (layer "F.Cu")
-    (at 72.092394 97.024 180)
+    (at 65.9 119.8 180)
     (descr "LED SMD 0603 (1608 Metric), square (rectangular) end terminal, IPC_7351 nominal, (Body size source: http://www.tortai-tech.com/upload/download/2011102023233369053.pdf), generated with kicad-footprint-generator")
     (tags "diode")
@@
   )
   (module "Resistor_SMD:R_0402_1005Metric" (layer "F.Cu")
-    (at 75.192394 94.524 90)
+    (at 69 117.3 90)
     (descr "Resistor SMD 0402 (1005 Metric), square (rectangular) end terminal, IPC_7351 nominal, (Body size source: http://www.tortai-tech.com/upload/download/2011102023233369053.pdf), generated with kicad-footprint-generator")
     (tags "resistor")
@@
   )
   (module "Package_TO_SOT_SMD:SOT-353_SC-70-5" (layer "F.Cu")
-    (at 74.992394 91.424 -90)
+    (at 68.8 114.2 -90)
     (descr "SOT-353, SC-70-5")
     (tags "SOT-353 SC-70-5")
@@
   )
   (module "Capacitor_SMD:C_0402_1005Metric" (layer "F.Cu")
-    (at 125 62.6 180)
+    (at 125.2 62.6 180)
     (descr "Capacitor SMD 0402 (1005 Metric), square (rectangular) end terminal, IPC_7351 nominal, (Body size source: IPC-SM-782 page 76, https://www.pcb-3d.com/wordpress/wp-content/uploads/ipc-sm-782a_amendment_1_and_2.pdf), generated with kicad-footprint-generator")
     (tags "capacitor")
@@
   )
   (module "TestPoint:TestPoint_Pad_2.0x2.0mm" (layer "B.Cu")
-    (at 75.804 94.224)
+    (at 69.611606 117)
     (descr "SMD rectangular pad as test Point, square 2.0mm side length")
     (tags "test point SMD pad rectangle square")
@@
   )
   (module "TestPoint:TestPoint_Pad_2.0x2.0mm" (layer "B.Cu")
-    (at 72.492394 94.224)
+    (at 66.3 117)
     (descr "SMD rectangular pad as test Point, square 2.0mm side length")
     (tags "test point SMD pad rectangle square")
@@
     (effects (font (size 1.5 1.5) (thickness 0.3)))
   )
+  (gr_text "Place jumpers and buttons here ->" (at 90.8 84.6) (layer "F.Cu")
+    (effects (font (size 1.5 1.5) (thickness 0.3)))
+  )
   (gr_text "NB uSDCARD \nonly used for \nCM4 modules \nwithout eMMC" (at 153.7025 96.879999 270) (layer "B.SilkS")
     (effects (font (size 1 1) (thickness 0.15)) (justify mirror))
@@
   (via (at 146 66) (size 0.45) (drill 0.25) (layers "F.Cu" "B.Cu") (net 8))
   (via (at 141.6 67.8) (size 0.45) (drill 0.25) (layers "F.Cu" "B.Cu") (net 8))
+  (segment (start 124.495 58.685) (end 124.58 58.6) (width 1) (layer "F.Cu") (net 9))
+  (via (at 122.6 56.6) (size 0.45) (drill 0.25) (layers "F.Cu" "B.Cu") (net 9))
+  (via (at 122.6 59.8) (size 0.45) (drill 0.25) (layers "F.Cu" "B.Cu") (net 9))
+  (via (at 122.6 58.6) (size 0.45) (drill 0.25) (layers "F.Cu" "B.Cu") (net 9))
+  (via (at 122.6 57.6) (size 0.45) (drill 0.25) (layers "F.Cu" "B.Cu") (net 9))
+  (via (at 122.6 61) (size 0.45) (drill 0.25) (layers "F.Cu" "B.Cu") (net 9))
+  (via (at 122.6 63.8) (size 0.45) (drill 0.25) (layers "F.Cu" "B.Cu") (net 9))
+  (via (at 122.6 64.8) (size 0.45) (drill 0.25) (layers "F.Cu" "B.Cu") (net 9))
+  (via (at 122.6 62.8) (size 0.45) (drill 0.25) (layers "F.Cu" "B.Cu") (net 9))
   (segment (start 137.68 68.505003) (end 137.549989 68.374992) (width 0.23) (layer "F.Cu") (net 12))
   (segment (start 137.68 69.880009) (end 138.600002 70.800011) (width 0.23) (layer "F.Cu") (net 12))
@@
   (segment (start 138.950013 70.45) (end 138.600002 70.800011) (width 0.23) (layer "B.Cu") (net 12))
   (segment (start 139.6 70.45) (end 138.950013 70.45) (width 0.23) (layer "B.Cu") (net 12))
+  (segment (start 125.68 62.6) (end 125.68 64.015) (width 1) (layer "F.Cu") (net 13))
+  (segment (start 125.68 64.015) (end 125.765 64.1) (width 1) (layer "F.Cu") (net 13))
   (zone (net 8) (net_name "Net-(C24-Pad1)") (layers "F.Cu" "In1.Cu" "In2.Cu" "B.Cu") (hatch full 0.508)
     (priority 1)
@@
       )
     )
+  )
+  (zone (net 9) (net_name "Net-(C28-Pad2)") (layers "F.Cu" "In1.Cu" "In2.Cu" "B.Cu") (hatch full 0.508)
+    (priority 1)
+    (connect_pads yes (clearance 0.3048))
+    (min_thickness 0.254)
+    (fill yes (thermal_gap 0) (thermal_bridge_width 0.254) (smoothing chamfer) (radius 0.381))
+    (polygon
+      (pts
+        (xy 125.2 65.2)
+        (xy 121.6 65.2)
+        (xy 121.6 55)
+        (xy 125.2 55)
+      )
+    )

Commit message: updating readme and some layout
Parts:
- removed C16, C50: 100uF, Capacitor_Tantalum_SMD:CP_EIA-7343-31_Kemet-D
- removed J11: USB_OTG, CM4IO:USB_Micro-B_EDAC_UCON00686
- C10, C11, C14, C15, C3, C4, C6, C7, C8, C9, R11, R12, R13, R14, R15, R16, R8, U13, Y1: moved to F.Cu
- C53, C54, C55, C56, J2, R31, U10: moved to B.Cu
- J3: value Conn_01x03 -> USB4085-GF-A_REVA; footprint Connector_PinHeader_2.54mm:PinHeader_1x03_P2.54mm_Vertical -> Open-HD:GCT_USB4085-GF-A_REVA
- JP1, JP2: footprint Jumper:SolderJumper-2_P1.3mm_Bridged_RoundedPad1.0x1.5mm -> Jumper:SolderJumper-2_P1.3mm_Open_Pad1.0x1.5mm
- JP3: footprint Jumper:SolderJumper-3_P1.3mm_Bridged12_RoundedPad1.0x1.5mm -> Jumper:SolderJumper-3_P1.3mm_Open_Pad1.0x1.5mm
- SW1: footprint Button_Switch_SMD:SW_SPST_B3S-1000 -> Button_Switch_SMD:SW_Push_SPST_NO_Alps_SKRK
- moved R31 121.8 mm to (142.2, 125.4), turned to -90 degrees
- moved C55 119.7 mm to (142.6, 132.2), turned to 180 degrees
- moved C53 119.7 mm to (142.6, 134.2), turned to 180 degrees
- moved U10 115.9 mm to (144.4, 125.0), turned to -90 degrees
- moved C54 115.2 mm to (142.6, 128.2), turned to 180 degrees
- moved C56 115.2 mm to (142.6, 130.2), turned to 180 degrees
- moved JP1 85.8 mm to (157.2, 87.0), turned to 90 degrees
- moved SW1 83.2 mm to (157.2, 82.4), turned to -90 degrees
- moved JP3 79.3 mm to (157.2, 91.2), turned to 90 degrees
- moved J3 79.2 mm to (155.4, 132.2), turned to 90 degrees
- moved JP2 77.8 mm to (157.2, 98.4), turned to -90 degrees
- moved C19 64.8 mm to (190.7, 151.0)
- moved C21 61.6 mm to (190.7, 153.0), turned to 180 degrees
- moved R36 59.6 mm to (186.7, 153.5)
- moved U7 56.9 mm to (182.7, 152.0)
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Connections:
- R8 pad 1: Net-(J11-Pad1) -> Net-(R8-Pad1)
Routing:
- net GND: track 0.00 -> 5.24 mm
- net Net-(C29-Pad2): track 0.00 -> 5.11 mm
- net Net-(C26-Pad1): track 0.00 -> 1.54 mm
- net /+5v: vias 0 -> 15
- added copper zone on F.Cu, net /+5v
Other:
- board size 47 x 86 mm -> 47 x 88.8 mm
- board text removed: "Compute Module 4"
- board text removed: "Fit for 1.8v GPIO"
- board text removed: "Fit for 3.3v GPIO"
- board text removed: "J3 : nBT_Dis GND"
- board text removed: "NB uSDCARD only used for CM4 modules without eMMC"
- board text removed: "nWireless_Dis"
- board text removed: "uSDCARD"

Commit message: started routing USB, added usb power switches, routing some USB-C
Parts:
- removed H1, H2, H3, H4, H5, H6, H7, H8: MountingHole, MountingHole:MountingHole_2.7mm_M2.5
- removed TP3, TP5: TestPoint, TestPoint:TestPoint_Pad_2.0x2.0mm
- removed U5: 74LVC1G07SE-7, Package_TO_SOT_SMD:SOT-353_SC-70-5
- added J4: 2199119-4, Open-HD:TE_2199119-4, F.Cu at (91.8, 93.3)
- added R20: 5.1k, Resistor_SMD:R_0402_1005Metric, F.Cu at (149.8, 134.3)
- added R22: 5.1k, Resistor_SMD:R_0402_1005Metric, B.Cu at (154.7, 130.9)
- C10, C11, C48, R12, R13, R16: moved to B.Cu
- C17, C19, C2, C20, C21, R36, U4, U6, U7: moved to F.Cu
- Y1: value 24MHz -> ECS-240-18-33-JGN-TR; footprint Crystal:Crystal_SMD_HC49-SD -> Open-HD:XTAL_ECS-240-18-33-JGN-TR
- moved C48 153.9 mm to (119.3, 127.8)
- moved R36 84.9 mm to (103.8, 134.9), turned to -90 degrees
- moved C12 77.1 mm to (122.7, 59.5), turned to 0 degrees
- moved C21 75.4 mm to (117.8, 133.9)
- moved C19 74.5 mm to (117.8, 135.7)
- moved U12 73.8 mm to (123.2, 62.0), turned to 0 degrees
- moved C20 73.2 mm to (121.5, 133.0), turned to 0 degrees
- moved C17 73.2 mm to (121.5, 131.2), turned to 0 degrees
- moved C13 70.5 mm to (120.8, 61.4)
- moved U7 68.3 mm to (117.7, 130.9)
- moved C2 63.2 mm to (117.6, 127.8), turned to 180 degrees
- moved C4 44.0 mm to (140.6, 128.6), turned to 0 degrees
- moved C14 41.1 mm to (140.6, 132.5)
- moved R8 40.2 mm to (147.3, 127.6), turned to 180 degrees
- moved C11 37.3 mm to (132.3, 125.8), turned to 90 degrees
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Connections:
- J3 pad A1: Net-(J3-PadA1) -> GND
- J3 pad A12: Net-(J3-PadA1) -> GND
- J3 pad A6: Net-(J3-PadA6) -> /USB2-HUB/USBD_P
- J3 pad A7: Net-(J3-PadA7) -> /USB2-HUB/USBD_N
- J3 pad B1: Net-(J3-PadA1) -> GND
- J3 pad B12: Net-(J3-PadA1) -> GND
- J3 pad B6: Net-(J3-PadB6) -> /USB2-HUB/USBD_P
- J3 pad B7: Net-(J3-PadB7) -> /USB2-HUB/USBD_N
- J3 pad P1: Net-(J3-PadP1) -> GND
- J3 pad P2: Net-(J3-PadP1) -> GND
- J3 pad P3: Net-(J3-PadP1) -> GND
- J3 pad P4: Net-(J3-PadP1) -> GND
- JP3 pad 1: /CM4_GPIO ( Ethernet, GPIO, SDCARD)/BT_nDis -> /CM4_GPIO ( Ethernet, GPIO, SDCARD)/WL_nDis
- JP3 pad 3: /CM4_GPIO ( Ethernet, GPIO, SDCARD)/WL_nDis -> /CM4_GPIO ( Ethernet, GPIO, SDCARD)/BT_nDis
- R10 pad 2: Net-(R10-Pad2) -> GND
- Y1 pad 2: Net-(C9-Pad1) -> GND
Routing:
- net /CM4_GPIO ( Ethernet, GPIO, SDCARD)/SD_DAT1: track 0.00 -> 26.7 mm, vias 0 -> 1
- net /CM4_GPIO ( Ethernet, GPIO, SDCARD)/SD_DAT0: track 0.00 -> 25.0 mm, vias 0 -> 1
- net /CM4_GPIO ( Ethernet, GPIO, SDCARD)/SD_CLK: track 0.00 -> 22.3 mm, vias 0 -> 1
- net /CM4_GPIO ( Ethernet, GPIO, SDCARD)/SD_DAT3: track 0.00 -> 19.2 mm, vias 0 -> 1
- net /CM4_GPIO ( Ethernet, GPIO, SDCARD)/SD_DAT2: track 0.00 -> 19.0 mm, vias 0 -> 1
- net /USB2-HUB/HD1_P: track 0.00 -> 16.5 mm
- net /USB2-HUB/HD1_N: track 0.00 -> 16.5 mm
- net /USB2-HUB/HD4_P: track 0.00 -> 13.9 mm
- net /USB2-HUB/HD4_N: track 0.00 -> 13.9 mm
- net Net-(J3-PadA4): track 0.00 -> 13.0 mm
- net /+3.3v: track 0.00 -> 11.5 mm, vias 0 -> 2
- net /USB2-HUB/HD2_P: track 0.00 -> 9.03 mm
- net /USB2-HUB/HD2_N: track 0.00 -> 9.03 mm
- net Net-(C9-Pad1): track 0.00 -> 9.02 mm
- net /USB2-HUB/USBD_N: track 0.00 -> 8.15 mm
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- added copper zone on F.Cu, net /USB2-HUB/VBUS_HP
- added copper zone on B.Cu, net /USB2-HUB/VBUS_LP
Other:
- outline, holes or cut-outs redrawn
- board text added: "<- Place jumpers and buttons here"
- board text removed: "Ext PSU"
- board text removed: "Place jumpers and buttons here ->"
